Commit message: visualization and pybullet simulator

File: assets/ground.urdf (robot description, URDF)
Before this commit: robot urdf_robot, 1 links, 0 joints
Links:
- removed link base_link
- added link baseLink, mass 0.0; collision box size=100 100 0.1; visual box size=100 100 0.1

Commit message: tuning

File: assets/ground.urdf (robot description, URDF)
Before this commit: robot ground, 1 links, 0 joints
Links:
- link baseLink: geometry collision box size=10 10 0.1; visual box size=10 10 0.1

Commit message: clean up folder

File: assets/ground.urdf (robot description, URDF)
Before this commit: robot ground, 1 links, 0 joints
Links:
- link baseLink: geometry collision box size=20 20 0.1; visual box size=20 20 0.1

Commit message: training model for maze

File: assets/ground.urdf (robot description, URDF)
Before this commit: robot ground, 1 links, 0 joints
Links:
- link baseLink: geometry collision box size=30 30 0.1; visual box size=30 30 0.1
